File: hw/WSPR-ease.kicad_sch (KiCad schematic)
At the start: 55 parts, among them J101 SMA, J102 pwr+data, J103 SMA, Q101 MMBF170, U101 GNSS module, U102 ESP32-S3-WROOM-1-N8R8, U103 SRV05-4, U104 TPS74612PQWDRBRQ1, U105 TPS22918DBVR, U106 LMR51430YDDCR

Commit message: Use relays and do layout over again to make these damned things fit
Parts:
- removed Q101: MMBF170, Package_TO_SOT_SMD:SOT-23, symbol Transistor_FET:BS170F
- removed R103, R104, R105, R106: 22, Resistor_SMD:R_0402_1005Metric, symbol Device:R_Small_US
- added Q101: 2N7002H, Package_TO_SOT_SMD:SOT-23, symbol Transistor_FET:2N7002H
- BT101: value CR2032 holder -> CR3032 holder; label CR2032 holder -> GNSS backup CR2032
Connections:
- net +3.3V: now also Q101.1 (G)
- net D+: now also U103.1 (IO1); no longer U103.3 (IO2)
- net D-: now also U103.3 (IO2); no longer U103.1 (IO1)
- net hiON: now also U102.7 (IO7)
- net loON: now also U102.5 (IO5)
- net at C101.1, R101.2, R102.1: now also Q101.2 (S)
- net at U102.12 (IO8): now also Q101.3 (D)
- net midON: now reaches U102.6 (IO6)
- no-connect marks 23 -> 24
Other:
- sheet Low Pass Filters ports: added midON; removed lo1ON, lo2ON
