File: hw/LPFs.kicad_sch (KiCad schematic)
At the start: 30 parts, among them K201 G6K-2, K202 G6K-2, K203 G6K-2, Q201 MMBF170, Q202 MMBF170, Q203 MMBF170

Commit message: Now using RP2040 as a DDS. I can use SPI co-host to program its (SPI) flash. I can use I2C between ESP32 and RP2040 to send commands and receive status.
Parts:
- C201, C204: value 910pF NP0 100V -> 910pF NP0 50V; footprint Capacitor_SMD:C_0603_1608Metric -> Capacitor_SMD:C_0402_1005Metric; LCSC C2941944 -> (none); MFG muRata -> (none); MPN GCM1885C2A911FA16D -> (none); Mouser_PN 81-GCM1885C2A911FA6D -> (none)
- C202, C203: value 1.6nF NP0 63V -> 1.6nF NP0 25V; footprint Capacitor_SMD:C_0603_1608Metric -> Capacitor_SMD:C_0402_1005Metric; LCSC C7471455 -> (none); MFG muRata -> (none); MPN GCM1885C1J162JA16D -> (none); Mouser_PN 81-GCM1885C1J162JA6D -> (none)
- C205, C208: footprint Capacitor_SMD:C_0603_1608Metric -> Capacitor_SMD:C_0402_1005Metric; LCSC C2176790 -> (none); MFG muRata -> (none); MPN GRM1885C1H331JA01D -> (none); Mouser_PN 81-GRM39C331J50 -> (none)
- C206, C207: footprint Capacitor_SMD:C_0603_1608Metric -> Capacitor_SMD:C_0402_1005Metric; LCSC C597173 -> (none); MFG muRata -> (none); MPN GRM1885C1H561JA01D -> (none); Mouser_PN 81-GRM39C561J50 -> (none)
- C209, C212: footprint Capacitor_SMD:C_0603_1608Metric -> Capacitor_SMD:C_0402_1005Metric; LCSC C314304 -> (none); MFG Kyocera AVX -> (none); MPN KGM15ACG1H820FT -> (none); Mouser_PN 581-KGM15ACG1H820FT -> (none)
- C210, C211: footprint Capacitor_SMD:C_0603_1608Metric -> Capacitor_SMD:C_0402_1005Metric; LCSC C440147 -> (none); MFG muRata -> (none); MPN GCM1885C2A181JA16D -> (none); Mouser_PN 81-GCM1885C2A181JA6D -> (none)
Changed lines of the file:
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@@
 			)
 		)
-		(property "Value" "910pF NP0 100V"
+		(property "Value" "910pF NP0 50V"
 			(at 137.16 60.706 0)
 			(effects
@@
 			)
 		)
-		(property "Footprint" "Capacitor_SMD:C_0603_1608Metric"
+		(property "Footprint" "Capacitor_SMD:C_0402_1005Metric"
 			(at 138.1252 62.23 0)
 			(effects
@@
 			)
 		)
-		(property "LCSC" "C2941944"
+		(property "LCSC" ""
 			(at 137.16 58.42 0)
 			(effects
@@
 			)
 		)
-		(property "MFG" "muRata"
+		(property "MFG" ""
 			(at 137.16 58.42 0)
 			(effects
@@
 			)
 		)
-		(property "MPN" "GCM1885C2A911FA16D"
+		(property "MPN" ""
 			(at 137.16 58.42 0)
 			(effects
@@
 			)
 		)
-		(property "Mouser_PN" "81-GCM1885C2A911FA6D "
+		(property "Mouser_PN" ""
 			(at 137.16 58.42 0)
 			(effects
@@
 			)
 		)
-		(property "Footprint" "Capacitor_SMD:C_0603_1608Metric"
+		(property "Footprint" "Capacitor_SMD:C_0402_1005Metric"
 			(at 83.5152 175.26 0)
 			(effects
@@
 			)
 		)
-		(property "LCSC" "C314304"
+		(property "LCSC" ""
 			(at 82.55 171.45 0)
 			(effects
@@
 			)
 		)
-		(property "MFG" "Kyocera AVX"
+		(property "MFG" ""
 			(at 82.55 171.45 0)
 			(effects
@@
 			)
 		)
-		(property "MPN" "KGM15ACG1H820FT "
+		(property "MPN" ""
 			(at 82.55 171.45 0)
 			(effects
@@
 			)
 		)
-		(property "Mouser_PN" "581-KGM15ACG1H820FT "
+		(property "Mouser_PN" ""
 			(at 82.55 171.45 0)
 			(effects
@@
 			)
 		)
-		(property "Footprint" "Capacitor_SMD:C_0603_1608Metric"
+		(property "Footprint" "Capacitor_SMD:C_0402_1005Metric"
 			(at 141.9352 116.84 0)
 			(effects
@@
 			)
 		)
-		(property "MFG" "muRata"
+		(property "MFG" ""
 			(at 140.97 113.03 0)
 			(effects
@@
 			)
 		)
-		(property "MPN" "GRM1885C1H331JA01D"
+		(property "MPN" ""
 			(at 140.97 113.03 0)
 			(effects
@@
 			)
 		)
-		(property "Mouser_PN" "81-GRM39C331J50 "
+		(property "Mouser_PN" ""
 			(at 140.97 113.03 0)
 			(effects
@@
 			)
 		)
-		(property "LCSC" "C2176790"
+		(property "LCSC" ""
 			(at 140.97 113.03 0)
 			(effects
@@
 			)
 		)
-		(property "Footprint" "Capacitor_SMD:C_0603_1608Metric"
+		(property "Footprint" "Capacitor_SMD:C_0402_1005Metric"
 			(at 121.6152 175.26 0)
 			(effects
@@
 			)
 		)
-		(property "LCSC" "C440147"
+		(property "LCSC" ""
 			(at 120.65 171.45 0)
 			(effects
@@
 			)
 		)
-		(property "MFG" "muRata"
+		(property "MFG" ""
 			(at 120.65 171.45 0)
 			(effects
@@
 			)
 		)
-		(property "MPN" "GCM1885C2A181JA16D"
+		(property "MPN" ""
 			(at 120.65 171.45 0)
 			(effects
@@
 			)
 		)
-		(property "Mouser_PN" "81-GCM1885C2A181JA6D"
+		(property "Mouser_PN" ""
 			(at 120.65 171.45 0)
 			(effects
@@
 			)
 		)
-		(property "Footprint" "Capacitor_SMD:C_0603_1608Metric"
+		(property "Footprint" "Capacitor_SMD:C_0402_1005Metric"
 			(at 103.8352 116.84 0)
 			(effects
@@
 			)
 		)
-		(property "MFG" "muRata"
+		(property "MFG" ""
 			(at 102.87 113.03 0)
 			(effects
@@
 			)
 		)
-		(property "MPN" "GRM1885C1H561JA01D"
+		(property "MPN" ""
 			(at 102.87 113.03 0)
 			(effects
@@
 			)
 		)
-		(property "Mouser_PN" "81-GRM39C561J50 "
+		(property "Mouser_PN" ""
 			(at 102.87 113.03 0)
 			(effects
@@
 			)
 		)
-		(property "LCSC" "C597173"
+		(property "LCSC" ""
 			(at 102.87 113.03 0)
 			(effects
@@
 			)
 		)
-		(property "Footprint" "Capacitor_SMD:C_0603_1608Metric"
+		(property "Footprint" "Capacitor_SMD:C_0402_1005Metric"
 			(at 122.8852 116.84 0)
 			(effects
@@
 			)
 		)
-		(property "MFG" "muRata"
+		(property "MFG" ""
 			(at 121.92 113.03 0)
 			(effects
@@
 			)
 		)
-		(property "MPN" "GRM1885C1H561JA01D"
+		(property "MPN" ""
 			(at 121.92 113.03 0)
 			(effects
@@
 			)
 		)
-		(property "Mouser_PN" "81-GRM39C561J50 "
+		(property "Mouser_PN" ""
 			(at 121.92 113.03 0)
 			(effects
@@
 			)
 		)
-		(property "LCSC" "C597173"
+		(property "LCSC" ""
 			(at 121.92 113.03 0)
 			(effects
@@
 			)
 		)
-		(property "Footprint" "Capacitor_SMD:C_0603_1608Metric"
+		(property "Footprint" "Capacitor_SMD:C_0402_1005Metric"
 			(at 140.6652 175.26 0)
 			(effects
@@
 			)
 		)
-		(property "LCSC" "C314304"
+		(property "LCSC" ""
 			(at 139.7 171.45 0)
 			(effects
@@
 			)
 		)
-		(property "MFG" "Kyocera AVX"
+		(property "MFG" ""
 			(at 139.7 171.45 0)
 			(effects
@@
 			)
 		)
-		(property "MPN" "KGM15ACG1H820FT "
+		(property "MPN" ""
 			(at 139.7 171.45 0)
 			(effects
@@
 			)
 		)
-		(property "Mouser_PN" "581-KGM15ACG1H820FT "
+		(property "Mouser_PN" ""
 			(at 139.7 171.45 0)
 			(effects
@@
 			)
 		)
-		(property "Value" "1.6nF NP0 63V"
+		(property "Value" "1.6nF NP0 25V"
 			(at 101.6 60.706 0)
 			(effects
@@
 			)
 		)
-		(property "Footprint" "Capacitor_SMD:C_0603_1608Metric"
+		(property "Footprint" "Capacitor_SMD:C_0402_1005Metric"
 			(at 102.5652 62.23 0)
 			(effects
@@
 			)
 		)
-		(property "LCSC" "C7471455"
+		(property "LCSC" ""
 			(at 101.6 58.42 0)
 			(effects
@@
 			)
 		)
-		(property "MFG" "muRata"
+		(property "MFG" ""
 			(at 101.6 58.42 0)
 			(effects
@@
 			)
 		)
-		(property "MPN" "GCM1885C1J162JA16D"
+		(property "MPN" ""
 			(at 101.6 58.42 0)
 			(effects
@@
 			)
 		)
-		(property "Mouser_PN" "81-GCM1885C1J162JA6D "
+		(property "Mouser_PN" ""
 			(at 101.6 58.42 0)
 			(effects
@@
 			)
 		)
-		(property "Value" "1.6nF NP0 63V"
+		(property "Value" "1.6nF NP0 25V"
 			(at 119.38 60.706 0)
 			(effects
@@
 			)
 		)
-		(property "Footprint" "Capacitor_SMD:C_0603_1608Metric"
+		(property "Footprint" "Capacitor_SMD:C_0402_1005Metric"
 			(at 120.3452 62.23 0)
 			(effects
@@
 			)
 		)
-		(property "LCSC" "C7471455"
+		(property "LCSC" ""
 			(at 119.38 58.42 0)
 			(effects
@@
 			)
 		)
-		(property "MFG" "muRata"
+		(property "MFG" ""
 			(at 119.38 58.42 0)
 			(effects
@@
 			)
 		)
-		(property "MPN" "GCM1885C1J162JA16D"
+		(property "MPN" ""
 			(at 119.38 58.42 0)
 			(effects
@@
 			)
 		)
-		(property "Mouser_PN" "81-GCM1885C1J162JA6D "
+		(property "Mouser_PN" ""
 			(at 119.38 58.42 0)
 			(effects
@@
 			)
 		)
-		(property "Footprint" "Capacitor_SMD:C_0603_1608Metric"
+		(property "Footprint" "Capacitor_SMD:C_0402_1005Metric"
 			(at 84.7852 116.84 0)
 			(effects
@@
 			)
 		)
-		(property "MFG" "muRata"
+		(property "MFG" ""
 			(at 83.82 113.03 0)
 			(effects
@@
 			)
 		)
-		(property "MPN" "GRM1885C1H331JA01D"
+		(property "MPN" ""
 			(at 83.82 113.03 0)
 			(effects
@@
 			)
 		)
-		(property "Mouser_PN" "81-GRM39C331J50 "
+		(property "Mouser_PN" ""
 			(at 83.82 113.03 0)
 			(effects
@@
 			)
 		)
-		(property "LCSC" "C2176790"
+		(property "LCSC" ""
 			(at 83.82 113.03 0)
 			(effects
@@
 			)
 		)
-		(property "Footprint" "Capacitor_SMD:C_0603_1608Metric"
+		(property "Footprint" "Capacitor_SMD:C_0402_1005Metric"
 			(at 102.5652 175.26 0)
 			(effects
@@
 			)
 		)
-		(property "LCSC" "C440147"
+		(property "LCSC" ""
 			(at 101.6 171.45 0)
 			(effects
@@
 			)
 		)
-		(property "MFG" "muRata"
+		(property "MFG" ""
 			(at 101.6 171.45 0)
 			(effects
@@
 			)
 		)
-		(property "MPN" "GCM1885C2A181JA16D"
+		(property "MPN" ""
 			(at 101.6 171.45 0)
 			(effects
@@
 			)
 		)
-		(property "Mouser_PN" "81-GCM1885C2A181JA6D"
+		(property "Mouser_PN" ""
 			(at 101.6 171.45 0)
 			(effects
@@
 			)
 		)
-		(property "Value" "910pF NP0 100V"
+		(property "Value" "910pF NP0 50V"
 			(at 83.82 60.706 0)
 			(effects
@@
 			)
 		)
-		(property "Footprint" "Capacitor_SMD:C_0603_1608Metric"
+		(property "Footprint" "Capacitor_SMD:C_0402_1005Metric"
 			(at 84.7852 62.23 0)
 			(effects
@@
 			)
 		)
-		(property "LCSC" "C2941944"
+		(property "LCSC" ""
 			(at 83.82 58.42 0)
 			(effects
@@
 			)
 		)
-		(property "MFG" "muRata"
+		(property "MFG" ""
 			(at 83.82 58.42 0)
 			(effects
@@
 			)
 		)
-		(property "MPN" "GCM1885C2A911FA16D"
+		(property "MPN" ""
 			(at 83.82 58.42 0)
 			(effects
@@
 			)
 		)
-		(property "Mouser_PN" "81-GCM1885C2A911FA6D "
+		(property "Mouser_PN" ""
 			(at 83.82 58.42 0)
 			(effects
