File: hw/LPFs.kicad_sch (KiCad schematic)
At the start: 30 parts, among them K201 G6K-2, K202 G6K-2, K203 G6K-2, Q201 MMBF170, Q202 MMBF170, Q203 MMBF170

Commit message: Switched to SI5351 clocking MACHXO2 CPLD to drive gate driver for MOSFETs. It passes DRC but needs serious reviewing.
Parts:
- Q201, Q202, Q203: value MMBF170 -> IRLML2060; LCSC C151058 -> (none); MFG Diodes inc -> Infineon; MPN MMBF170Q-13-F -> IRLML2060TRPBF; Mouser_PN 621-MMBF170Q-13-F -> 942-IRLML2060TRPBF
Other:
- title: Low Pass Filters -> Transmitter
Changed lines of the file:
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@@
 	(paper "USLetter")
 	(title_block
-		(title "Low Pass Filters")
-		(date "2025-11-24")
+		(title "Transmitter")
+		(date "2026-07-04")
 		(company "WB7NAB")
 	)
@@
 			)
 		)
-		(property "Value" "MMBF170"
+		(property "Value" "IRLML2060"
 			(at 62.738 175.514 0)
 			(effects
@@
 			)
 		)
-		(property "LCSC" "C151058"
+		(property "LCSC" ""
 			(at 71.12 171.45 0)
 			(effects
@@
 			)
 		)
-		(property "MFG" "Diodes inc"
+		(property "MFG" "Infineon"
 			(at 71.12 171.45 0)
 			(effects
@@
 			)
 		)
-		(property "MPN" "MMBF170Q-13-F"
+		(property "MPN" "IRLML2060TRPBF"
 			(at 71.12 171.45 0)
 			(effects
@@
 			)
 		)
-		(property "Mouser_PN" "621-MMBF170Q-13-F"
+		(property "Mouser_PN" "942-IRLML2060TRPBF"
 			(at 71.12 171.45 0)
 			(effects
@@
 			)
 		)
-		(property "Value" "MMBF170"
+		(property "Value" "IRLML2060"
 			(at 64.008 117.094 0)
 			(effects
@@
 			)
 		)
-		(property "LCSC" "C151058"
+		(property "LCSC" ""
 			(at 72.39 113.03 0)
 			(effects
@@
 			)
 		)
-		(property "MFG" "Diodes inc"
+		(property "MFG" "Infineon"
 			(at 72.39 113.03 0)
 			(effects
@@
 			)
 		)
-		(property "MPN" "MMBF170Q-13-F"
+		(property "MPN" "IRLML2060TRPBF"
 			(at 72.39 113.03 0)
 			(effects
@@
 			)
 		)
-		(property "Mouser_PN" "621-MMBF170Q-13-F"
+		(property "Mouser_PN" "942-IRLML2060TRPBF"
 			(at 72.39 113.03 0)
 			(effects
@@
 			)
 		)
-		(property "Value" "MMBF170"
+		(property "Value" "IRLML2060"
 			(at 65.278 62.484 0)
 			(effects
@@
 			)
 		)
-		(property "LCSC" "C151058"
+		(property "LCSC" ""
 			(at 73.66 58.42 0)
 			(effects
@@
 			)
 		)
-		(property "MFG" "Diodes inc"
+		(property "MFG" "Infineon"
 			(at 73.66 58.42 0)
 			(effects
@@
 			)
 		)
-		(property "MPN" "MMBF170Q-13-F"
+		(property "MPN" "IRLML2060TRPBF"
 			(at 73.66 58.42 0)
 			(effects
@@
 			)
 		)
-		(property "Mouser_PN" "621-MMBF170Q-13-F"
+		(property "Mouser_PN" "942-IRLML2060TRPBF"
 			(at 73.66 58.42 0)
 			(effects

Commit message: Various schematic clean ups. Improved/fixed decoupling around relays. Filter Vdd for TCXO and SI5351 to try to minimize modulation of the clock freq by noise
Parts:
- added C201, C206, C211: 1uF X5R 25V, Capacitor_SMD:C_0402_1005Metric, symbol Device:C
- renumbered C201 to C202, C202 to C203, C203 to C204, C204 to C205, C205 to C207, C206 to C208, C207 to C209, C208 to C210, C209 to C212, C210 to C213, C211 to C214, C212 to C215
Connections:
- net GND: now also C201.2, C206.2, C211.2
- net VBUS: now also C201.1, C206.1, C211.1
