File: hw/WSPR-ease.kicad_pcb (KiCad board)
At the start: 4 copper layers, 99 x 64 mm, 182 parts, among them J101 pwr+data, J102 SMA, J103 SMA, J401 SJ1-3514-SMT-TR, K201 G6K-2, K202 G6K-2, K203 G6K-2, Q101 IRLML2060, Q201 IRLML2060, Q202 IRLML2060, Q203 IRLML2060, Q301 IRLML2060, Q302 IRLML2060, Q303 IRLML2060, Q304 IRLML2060, T301 BN-43-202_DualPri_CTSec, U101 TPS74612PQWDRBRQ1, U102 SRV05-4, U103 TPS22918DBVR, U104 ESP32-S3-WROOM-1-N8R8, U105 LMR51430YDDCR, U106 GNSS module, U107 AP2112K-3.3TRG1, U301 UCC27523DGN, U302 UCC27523DGN, U303 TPS62A02NDRL, U401 ICE40UP5K-SG48ITR, U402 TAA5242IRGER, U403 SI5351A-B-GT, Y401 40MHz

Commit message: Getting closer but not timing at 40MHz clock still. I think I have a fix but I have run out of time. Checkpoint.
Parts:
- moved R409 33.8 mm to (56.1, 98.2)
Connections:
- net /D+ renamed /USBD+
- net /D- renamed /USBD-
- net /Exciter/txco renamed /Exciter/tcxo
- U104 pad 25: unconnected-(U104-IO48-Pad25) -> /txI2Sdata
- U401 pad 18: unconnected-(U401B-IOB_31b-Pad18) -> /txBCLK
- U401 pad 19: unconnected-(U401B-IOB_29b-Pad19) -> /txSYNC
- U401 pad 6: unconnected-(U401B-IOB_13b-Pad6) -> /txI2Sdata
Routing:
- net /txI2Sdata: track 0.00 -> 27.7 mm, vias 0 -> 2
- net /txBCLK: track 11.0 -> 26.1 mm, vias 0 -> 2
- net /txSYNC: track 11.4 -> 25.2 mm, vias 0 -> 2
- net /fpgaMISO: track 27.1 -> 25.2 mm
- net /fpgaSCK: track 27.5 -> 25.7 mm
- net /fpgaMOSI: track 28.4 -> 26.6 mm
- net /fpgaNCS: track 28.0 -> 26.1 mm
- net /txSCL: track 41.0 -> 39.9 mm
- net /txSDA: track 42.1 -> 41.1 mm
- net /fpgaCRESET: track 40.0 -> 40.6 mm

Commit message: Clean up old garbage files
Parts:
- moved C203 4.69 mm to (107.1, 105.5), turned to -90 degrees
- moved C318 4.64 mm to (79.8, 90.2), turned to 180 degrees
- moved C307 3.61 mm to (76.0, 90.3)
- moved C212 3.26 mm to (113.7, 75.3), turned to -90 degrees
- moved C317 3.24 mm to (79.8, 91.2), turned to 180 degrees
- moved C202 2.88 mm to (110.9, 103.2), turned to -90 degrees
- moved C207 2.44 mm to (113.1, 87.0), turned to -90 degrees
- moved L204 2.31 mm to (111.2, 87.6)
- moved C316 1.86 mm to (79.8, 92.2), turned to 180 degrees
- moved C208 1.69 mm to (111.7, 90.1), turned to 0 degrees
- moved C305 1.61 mm to (77.0, 90.4)
- moved C314 1.15 mm to (79.8, 94.2), turned to 180 degrees
- moved C211 0.74 mm to (129.0, 72.4), turned to 0 degrees
- moved C315 0.63 mm to (79.8, 93.2), turned to 180 degrees
- moved C214 0.62 mm to (113.9, 80.1)
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- renumbered C104 to C101, C107 to C102, C110 to C103, C101 to C104, C102 to C105, C103 to C106, C105 to C107, C106 to C109, C109 to C110, C119 to C114, C120 to C115, C114 to C116, C115 to C117, C116 to C118, C117 to C119, C118 to C120, J102 to J101, J101 to J102, R104 to R101, R106 to R102, R102 to R103, R103 to R104, R101 to R105, R105 to R106, R109 to R107, R110 to R108, R111 to R109, R112 to R110, R113 to R111, R107 to R112, R108 to R113, U104 to U101, U101 to U104, U106 to U105, U107 to U106, U105 to U107
Connections:
- net /Exciter/FPGACLK renamed /Exciter/txCLK
- net /txBCLK renamed /modBCLK
- net /txI2Sdata renamed /modTxData
- net /txSYNC renamed /modSYNC
Routing:
- net /paEn: track 67.3 -> 70.5 mm
- net Net-(C208-Pad1): track 8.49 -> 5.88 mm
- net Net-(C213-Pad1): track 11.8 -> 10.4 mm
- net Net-(C212-Pad1): track 9.20 -> 7.89 mm
- net Net-(C202-Pad1): track 13.7 -> 12.7 mm
- net VBUS: track 95.1 -> 95.7 mm
- net GND: track 170.6 -> 170.5 mm, vias 317 -> 319
