File: hw/exciter.kicad_sch (KiCad schematic)
At the start: 22 parts, among them U401 LCMXO2-256HC-4SG32C, U402 SI5351A-B-GT, Y401 20MHz

Commit message: Various schematic clean ups. Improved/fixed decoupling around relays. Filter Vdd for TCXO and SI5351 to try to minimize modulation of the clock freq by noise
Parts:
- added C416: 1uF X5R 25V, Capacitor_SMD:C_0402_1005Metric, symbol Device:C
- added FB401: 600@1A, Inductor_SMD:L_0603_1608Metric, symbol Device:FerriteBead_Small
- added TP401: A, TestPoint:TestPoint_Pad_1.5x1.5mm, symbol Connector:TestPoint
- added TP402: B, TestPoint:TestPoint_Pad_1.5x1.5mm, symbol Connector:TestPoint
- renumbered C405 to C403, C406 to C404, C403 to C405, C404 to C406, C415 to C411, C416 to C412, C411 to C413, C417 to C414, C418 to C415, R404 to R402, R402 to R403, R403 to R404
Connections:
- net +3.3V: now also FB401.1; no longer C407.1, C408.1, C409.2, C410.2, C414.1, C415.1, U402.1 (VDD), U402.7 (VDDO), Y401.4 (VDD)
- net GND: now also C416.2
- net txSCL: now also R403.1; no longer R404.1
- net txSDA: now also R404.1; no longer R403.1
- net at U401.27 (SDA/PCLKC0_0): now also TP401.1
- net at U401.28 (SCL/PCLKT0_0): now also TP402.1
- new net +VDDA: C407.1, C408.1, C409.2, C410.2, C414.1, C415.1, C416.1, FB401.2, U402.1 (VDD), U402.7 (VDDO), Y401.4 (VDD)
- no-connect marks 13 -> 11
Other:
- moved on the sheet: R403, R404

Commit message: Simplify. Put exciter stuff onto transmitter sheet.
Parts:
- removed C401, C402, C403, C404, C405, C406, C409, C410, C411, C412, C413, C415: 100nF X7R 50V, Capacitor_SMD:C_0402_1005Metric, symbol Device:C
- removed C407, C408, C414, C416: 1uF X5R 25V, Capacitor_SMD:C_0402_1005Metric, symbol Device:C
- removed FB401: 600@1A, Inductor_SMD:L_0603_1608Metric, symbol Device:FerriteBead_Small
- removed R401, R402: 27, Resistor_SMD:R_0402_1005Metric, symbol Device:R_US
- removed R403, R404: 5.1k, Resistor_SMD:R_0402_1005Metric, symbol Device:R_US
- removed TP401: A, TestPoint:TestPoint_Pad_1.5x1.5mm, symbol Connector:TestPoint
- removed TP402: B, TestPoint:TestPoint_Pad_1.5x1.5mm, symbol Connector:TestPoint
- removed U401: LCMXO2-256HC-4SG32C, Package_DFN_QFN:QFN-32-1EP_5x5mm_P0.5mm_EP3.1x3.1mm_ThermalVias, symbol Library:LCMXO2-SG32
- removed U402: SI5351A-B-GT, Package_SO:MSOP-10_3x3mm_P0.5mm, symbol Oscillator:Si5351A-B-GT
- removed Y401: 20MHz, Library:ECSTXO201633400TR, symbol Library:ECS-TX-5032-200
Connections:
- no-connect marks 11 -> 0

Commit message: Prep to go back to FPGA. Board is routed except for power layer zones. No time to run DRC yet.
Parts:
- added C401, C402, C403, C405, C412, C414, C421, C425, C429, C430, C431, C433: 100nF X7R 50V, Capacitor_SMD:C_0402_1005Metric, symbol Device:C
- added C404, C407, C408, C413, C415, C422, C426: 4.7uF, Capacitor_SMD:C_0402_1005Metric, symbol Device:C
- added C406, C409: 10uF X5R 25V, Capacitor_SMD:C_0603_1608Metric, symbol Device:C
- added C410, C411, C416, C417, C418, C419, C420, C427, C428: 1uF X5R 25V, Capacitor_SMD:C_0402_1005Metric, symbol Device:C
- added C423: 1.6nF NP0 25V, Capacitor_SMD:C_0402_1005Metric, symbol Device:C
- added C424: 330pF NP0 50V, Capacitor_SMD:C_0402_1005Metric, symbol Device:C
- added C432: 1uF, Capacitor_SMD:C_0402_1005Metric, symbol Device:C
- added J402: SJ1-3514-SMT-TR, Library:35RASMT2BHWNTRX, symbol Library:35RASMT2BHWNTRX
- added R401: 100, Resistor_SMD:R_0402_1005Metric, symbol Device:R_Small_US
- added R402, R403, R410, R411: 5.1k, Resistor_SMD:R_0402_1005Metric, symbol Device:R_US
- added R404, R405, R408, R409: 10k, Resistor_SMD:R_0402_1005Metric, symbol Device:R_US
- added R406, R407: 27, Resistor_SMD:R_0402_1005Metric, symbol Device:R_US
- added TP401: A, TestPoint:TestPoint_Pad_1.5x1.5mm, symbol Connector:TestPoint
- added TP402: B, TestPoint:TestPoint_Pad_1.5x1.5mm, symbol Connector:TestPoint
- added U402: ICE40UP5K-SG48ITR, Package_DFN_QFN:QFN-48-1EP_7x7mm_P0.5mm_EP5.6x5.6mm, symbol Library:ICE40UP5K-SG48ITR
- added U403: TAA5242IRGER, Library:TAA5242IRGER, symbol Library:TAA5242IRGER
- added U404: SI5351A-B-GT, Package_SO:MSOP-10_3x3mm_P0.5mm, symbol Oscillator:Si5351A-B-GT
- added Y401: 40MHz, Library:ECSTXO201633400TR, symbol Library:ECS-TXO-2016-33-400-TR
Connections:
- new net: C405.2, C406.2, U403.1 (DREG)
- new net: C420.1, U403.24 (VREF)
- new net: C417.1, U403.16 (IN1M)
- new net: C419.1, U403.18 (IN2M)
- new net: TP402.1, U402.3 (IOB_9b)
- new net: TP401.1, U402.4 (IOB_8a)
- new net: C411.1, R402.2, U403.14 (MICBIAS)
- new net: C413.1, C414.2, R401.1, U402.29 (VCCPLL)
- new net: R407.2, U404.9 (CLK1)
- new net: C416.1, U403.15 (IN1P)
- new net: C418.1, U403.17 (IN2P)
- new net: C431.1, Y401.3 (OUTPUT)
- new net: C431.2, U404.2 (XA)
- new net: R406.2, U404.10 (CLK0)
- new net +3.3V: C409.2, R404.2, R410.2, R411.2, U403.6 (IOVDD)
- new net +VDDA: C410.1, C427.1, C428.1, C429.2, C430.2, C432.1, C433.1, U403.23 (AVDD), U404.1 (VDD), U404.7 (VDDO), Y401.1 (TRI-STATE), Y401.4 (VDD)
- new net +VFPGACORE: C402.2, C403.2, C407.1, C408.1, R401.2, U402.30 (VCC), U402.5 (VCC)
- new net +VFPGAIO: C401.2, C404.1, C412.2, C415.1, C421.2, C422.1, C425.2, C426.1, U402.1 (VCCIO_2), U402.22 (SPI_VCCIO1), U402.24 (VPP_2V5), U402.33 (VCCIO_0)
- new net FPGACLK: R406.1, U402.35 (IOT_46b_G0)
- new net GND: C401.1, C402.1, C403.1, C404.2, C405.1, C406.1, C407.2, C408.2, C409.1, C410.2, C411.2, C412.1, C413.2, C414.1, C415.2, C417.2, C418.2, C419.2, C420.2, C421.1, C422.2, C423.2, C424.2, C425.1, C426.2, C427.2, C428.2, C429.1, C430.1, C432.2, C433.2, J402.1 (R), R408.2, R409.2, U402.49 (GND), U403.10 (MD4), U403.12 (MD5), U403.13 (MD0), U403.19 (VSSA_1), U403.20 (VSSA_2), U403.21 (VSSA_3), U403.22 (VSSA_4), U403.25 (EP), U403.26 (VSS_1), U403.27 (VSS_2), U403.28 (VSS_3), U403.29 (VSS_4), U403.5 (MD6), U403.7 (MD1), U403.8 (MD2), U403.9 (MD3), U404.8 (GND), Y401.2 (GND)
- new net amPWM: R403.2, U402.46 (IOB_0a)
- new net amTracking: C423.1, R403.1
- new net fpgaCRESET: R409.1, U402.8 (~{CRESET})
- new net fpgaDONE: U402.7 (CDONE)
- new net fpgaMISO: U402.14 (IOB_32a_SPI_SO)
- new net fpgaMOSI: U402.17 (IOB_33b_SPI_SI)
- new net fpgaNCS: U402.16 (IOB_35b_SPI_SS)
- new net fpgaNRESET: U402.36 (IOT_48b)
- new net fpgaSCLK: U402.15 (IOB_34a_SPI_SCK)
- new net gnssPPS: U402.25 (IOT_36b)
- new net keyerDahPTT: J402.2 (S), R404.1
- new net keyerDit: C424.1, R405.1
- new net micBCLK: U403.2 (BCLK)
- new net micDOUT: U403.4 (DOUT)
- new net micSYNC: U403.3 (FSYNC)
- new net micTip: C416.2, J402.3 (T), R402.1, R405.2
- new net nPullBase: U402.45 (IOB_5b)
- new net nPullPeak: U402.48 (IOB_4a)
- new net nPushBase: U402.42 (IOT_51a)
- new net nPushPeak: U402.37 (IOT_45a_G1)
- new net paEn: R408.1, U402.47 (IOB_2a)
- new net txSCL: R410.1, U404.4 (SCL)
- new net txSDA: R411.1, U404.5 (SDA)
- new net txco: R407.1, U402.44 (IOB_3b_G6)
- no-connect marks 0 -> 25

Commit message: Now we pass schematic and PCB DRC and 3D renders nicely also.
Parts:
- U401: renamed from U402; footprint Package_DFN_QFN:QFN-48-1EP_7x7mm_P0.5mm_EP5.6x5.6mm -> Library:QFN50P700X700X100-49N-D
- renumbered J402 to J401, R404 to R403, R403 to R404, U403 to U402, U404 to U403
Connections:
- net keyerDahPTT renamed micSleeve
- no-connect marks 25 -> 26
Other:
- moved on the sheet: C432, C433, Y401

Commit message: Remove old stuff, describe new FPGA strategy, clean up schematic to show this more cleanly, add I2S I/O for ESP32 to FPGA and mic ADC with common clocking.
Connections:
- net micBCLK is gone; now on net txBCLK: U402.2 (BCLK)
- net micSYNC is gone; now on net txSYNC: U402.3 (FSYNC)
- net txBCLK: now reaches U401.10 (IOB_18a)
- net txI2Sdata: now reaches U401.6 (IOB_13b)
- net txSYNC: now reaches U401.9 (IOB_16a)
- no-connect marks 26 -> 23
Changed lines of the file:
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@@
-	)
-	(no_connect
-		(at 88.9 106.68)
 	)
 	(no_connect
@@
 	)
 	(no_connect
-		(at 88.9 104.14)
-	)
-	(no_connect
 		(at 69.85 38.1)
 	)
@@
 	)
 	(no_connect
-		(at 88.9 109.22)
-	)
-	(no_connect
 		(at 88.9 127)
 	)
@@
 	(wire
 		(pts
+			(xy 88.9 109.22) (xy 90.17 109.22)
+		)
+		(stroke
+			(width 0)
+			(type default)
+		)
+	)
+	(wire
+		(pts
 			(xy 71.12 68.58) (xy 69.85 68.58)
 		)
@@
 	(wire
 		(pts
+			(xy 88.9 106.68) (xy 90.17 106.68)
+		)
+		(stroke
+			(width 0)
+			(type default)
+		)
+	)
+	(wire
+		(pts
 			(xy 232.41 88.9) (xy 234.95 88.9)
 		)
@@
 		(pts
 			(xy 151.13 158.75) (xy 151.13 157.48)
+		)
+		(stroke
+			(width 0)
+			(type default)
+		)
+	)
+	(wire
+		(pts
+			(xy 88.9 104.14) (xy 90.17 104.14)
 		)
 		(stroke
@@
 		)
 	)
+	(hierarchical_label "txBCLK"
+		(shape input)
+		(at 90.17 109.22 0)
+		(effects
+			(font
+				(size 1.27 1.27)
+			)
+			(justify left)
+		)
+	)
 	(hierarchical_label "fpgaDONE"
 		(shape output)
@@
 		)
 	)
+	(hierarchical_label "txI2Sdata"
+		(shape input)
+		(at 90.17 104.14 0)
+		(effects
+			(font
+				(size 1.27 1.27)
+			)
+			(justify left)
+		)
+	)
 	(hierarchical_label "nPullBase"
 		(shape input)
@@
 		)
 	)
-	(hierarchical_label "micBCLK"
+	(hierarchical_label "txBCLK"
 		(shape input)
 		(at 254 73.66 0)
@@
 		)
 	)
+	(hierarchical_label "txSYNC"
+		(shape input)
+		(at 90.17 106.68 0)
+		(effects
+			(font
+				(size 1.27 1.27)
+			)
+			(justify left)
+		)
+	)
 	(hierarchical_label "txSCL"
 		(shape input)
@@
 		)
 	)
-	(hierarchical_label "micSYNC"
+	(hierarchical_label "txSYNC"
 		(shape input)
 		(at 254 71.12 0)

Commit message: Getting closer but not timing at 40MHz clock still. I think I have a fix but I have run out of time. Checkpoint.
Connections:
- net txBCLK: now also U401.18 (IOB_31b); no longer U401.10 (IOB_18a)
- net txSYNC: now also U401.19 (IOB_29b); no longer U401.9 (IOB_16a)
- net txco renamed tcxo
Changed lines of the file:
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@@
+	)
+	(no_connect
+		(at 88.9 106.68)
 	)
 	(no_connect
@@
 	)
 	(no_connect
-		(at 88.9 124.46)
-	)
-	(no_connect
 		(at 88.9 119.38)
 	)
@@
 	)
 	(no_connect
+		(at 88.9 109.22)
+	)
+	(no_connect
 		(at 88.9 116.84)
 	)
@@
 	)
 	(no_connect
-		(at 88.9 127)
-	)
-	(no_connect
 		(at 252.73 64.77)
 	)
@@
 	(wire
 		(pts
-			(xy 88.9 109.22) (xy 90.17 109.22)
-		)
-		(stroke
-			(width 0)
-			(type default)
-		)
-	)
-	(wire
-		(pts
 			(xy 71.12 68.58) (xy 69.85 68.58)
 		)
@@
 	(wire
 		(pts
+			(xy 88.9 127) (xy 90.17 127)
+		)
+		(stroke
+			(width 0)
+			(type default)
+		)
+	)
+	(wire
+		(pts
 			(xy 208.28 63.5) (xy 208.28 64.77)
 		)
@@
 	(wire
 		(pts
-			(xy 88.9 106.68) (xy 90.17 106.68)
-		)
-		(stroke
-			(width 0)
-			(type default)
-		)
-	)
-	(wire
-		(pts
 			(xy 232.41 88.9) (xy 234.95 88.9)
 		)
@@
 		(pts
 			(xy 217.17 60.96) (xy 201.93 60.96)
+		)
+		(stroke
+			(width 0)
+			(type default)
+		)
+	)
+	(wire
+		(pts
+			(xy 88.9 124.46) (xy 90.17 124.46)
 		)
 		(stroke
@@
 		)
 	)
-	(label "txco"
+	(label "tcxo"
 		(at 142.24 179.07 0)
 		(effects
@@
 		)
 	)
-	(label "txco"
+	(label "tcxo"
 		(at 228.6 152.4 0)
 		(effects
@@
 	(hierarchical_label "txBCLK"
 		(shape input)
-		(at 90.17 109.22 0)
+		(at 90.17 127 0)
 		(effects
 			(font
@@
 	(hierarchical_label "txSYNC"
 		(shape input)
-		(at 90.17 106.68 0)
-		(effects
-			(font
+		(at 90.17 124.46 0)
+		(effects
+			(font

Commit message: Clean up old garbage files
Connections:
- net FPGACLK renamed txCLK
- net fpgaSCLK renamed fpgaSCK
- net txBCLK renamed modBCLK
- net txI2Sdata renamed modTxData
- net txSYNC renamed modSYNC
Changed lines of the file:
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@@
 		)
 	)
-	(label "FPGACLK"
+	(label "txCLK"
 		(at 142.24 173.99 0)
 		(effects
@@
 		)
 	)
-	(label "FPGACLK"
+	(label "txCLK"
 		(at 71.12 58.42 0)
 		(effects
@@
 		)
 	)
-	(hierarchical_label "txBCLK"
+	(hierarchical_label "modBCLK"
 		(shape input)
 		(at 90.17 127 0)
@@
 		)
 	)
-	(hierarchical_label "txI2Sdata"
+	(hierarchical_label "modTxData"
 		(shape input)
 		(at 90.17 104.14 0)
@@
 		)
 	)
-	(hierarchical_label "fpgaSCLK"
+	(hierarchical_label "fpgaSCK"
 		(shape input)
 		(at 90.17 134.62 0)
@@
 		)
 	)
-	(hierarchical_label "txBCLK"
+	(hierarchical_label "modBCLK"
 		(shape input)
 		(at 254 73.66 0)
@@
 		)
 	)
-	(hierarchical_label "txSYNC"
+	(hierarchical_label "modSYNC"
 		(shape input)
 		(at 90.17 124.46 0)
@@
 		)
 	)
-	(hierarchical_label "txSYNC"
+	(hierarchical_label "modSYNC"
 		(shape input)
 		(at 254 71.12 0)
